Commit message: Rebase from 'upstream'

File: orbbec_description/urdf/astra2.urdf.xacro (robot description, xacro)
@@ -3,25 +3,25 @@
      Commit Version: 1.6.0-4-g7f85cfe  Build Version: 1.6.7995.38578
      For more information, please see http://wiki.ros.org/sw_urdf_exporter -->
-<robot xmlns:xacro="http://ros.org/wiki/xacro" name="gemini2">
-    <xacro:property name="mesh_path" value="package://orbbec_description/meshes/gemini2/" />
+<robot xmlns:xacro="http://ros.org/wiki/xacro" name="astra2">
+    <xacro:property name="mesh_path" value="package://orbbec_description/meshes/astra2/" />
   <link
     name="camera_link">
     <inertial>
       <origin
-        xyz="0.0027714370634978 -9.29434319373592E-06 0.0128014057830239"
-        rpy="0 0 0" />
-      <mass
-        value="0.0186201988654731" />
-      <inertia
-        ixx="1.38952652762223E-05"
-        ixy="-4.88105621547421E-09"
-        ixz="1.98670223779875E-08"
-        iyy="1.7072236178685E-06"
-        iyz="-8.49860443053716E-09"
-        izz="1.31795237727551E-05" />
-    </inertial>
-    <visual>
-      <origin
-        xyz="0 0 0"
+        xyz="-0.0160938085585399 -0.00100885505248632 0.0279919581775268"
+        rpy="0 0 0" />
+      <mass
+        value="0.0101524380243699" />
+      <inertia
+        ixx="1.69184979927567E-05"
+        ixy="-8.18066547859061E-09"
+        ixz="-1.27426373196599E-09"
+        iyy="7.7096717121366E-07"
+        iyz="1.08838945581987E-08"
+        izz="1.61801971464778E-05" />
+    </inertial>
+    <visual>
+      <origin
+        xyz="-0.012323995999904 -0.0374999999985815 -0.0281503197112"
         rpy="0 0 0" />
       <geometry>
@@ -32,5 +32,5 @@
         name="">
         <color
-          rgba="0.792156862745098 0.819607843137255 0.933333333333333 1" />
+          rgba="0.827450980392157 0.698039215686274 0.490196078431373 1" />
       </material>
     </visual>
@@ -46,45 +46,98 @@
   </link>
   <link
-    name="camera_botter_screw_frame">
-    <inertial>
-      <origin
-        xyz="0.00255175353418556 -0.00123907270798541 0.0118889783016768"
-        rpy="0 0 0" />
-      <mass
-        value="0.00564464822744556" />
-      <inertia
-        ixx="3.07688942133184E-06"
-        ixy="-1.84968755859098E-08"
-        ixz="-9.2787127214088E-09"
-        iyy="2.27625032346061E-07"
-        iyz="1.65176768024159E-08"
-        izz="2.93984854119768E-06" />
-    </inertial>
-    <visual>
-      <origin
-        xyz="0 0 0"
-        rpy="0 0 0" />
-      <geometry>
-        <mesh
-          filename="${mesh_path}camera_botter_screw_frame.STL" />
-      </geometry>
-      <material
-        name="">
-        <color
-          rgba="0.792156862745098 0.819607843137255 0.933333333333333 1" />
-      </material>
-    </visual>
-    <collision>
-      <origin
-        xyz="0 0 0"
-        rpy="0 0 0" />
-      <geometry>
-        <mesh
-          filename="${mesh_path}camera_botter_screw_frame.STL" />
-      </geometry>
-    </collision>
-  </link>
-  <joint
-    name="camera_botter_screw_frame"
+    name="camera_bottom_screw_frame">
+    <inertial>
+      <origin
+        xyz="-0.00635589512085941 1.59480886486103E-08 0.0118534361269284"
+        rpy="0 0 0" />
+      <mass
+        value="0.00583601107155577" />
+      <inertia
+        ixx="3.65092579901689E-06"
+        ixy="-5.00479838523244E-12"
+        ixz="7.68810468643615E-07"
+        iyy="2.03966087595316E-06"
+        iyz="6.18841137398479E-13"
+        izz="3.65126403038314E-06" />
+    </inertial>
+    <visual>
+      <origin
+        xyz="0 0 0"
+        rpy="0 0 0" />
+      <geometry>
+        <mesh
+          filename="${mesh_path}camera_bottom_screw_frame.STL" />
+      </geometry>
+      <material
+        name="">
+        <color
+          rgba="0.266666666666667 0.266666666666667 0.266666666666667 1" />
+      </material>
+    </visual>
+    <collision>
+      <origin
+        xyz="0 0 0"
+        rpy="0 0 0" />
+      <geometry>
+        <mesh
+          filename="${mesh_path}camera_bottom_screw_frame.STL" />
+      </geometry>
+    </collision>
+  </link>
+  <joint
+    name="camera_bottom_screw_frame"
+    type="fixed">
+    <origin
+      xyz="-0.012323995999904 -0.0374999999985815 -0.0281503197112"
+      rpy="0 0 0" />
+    <parent
+      link="camera_link" />
+    <child
+      link="camera_bottom_screw_frame" />
+    <axis
+      xyz="0 0 0" />
+  </joint>
+  <link
+    name="camera_ir_frame">
+    <inertial>
+      <origin
+        xyz="-0.00168460453866946 5.33451517362171E-07 6.08796009742363E-07"
+        rpy="0 0 0" />
+      <mass
+        value="0.000608348661221201" />
+      <inertia
+        ixx="6.79778952271057E-09"
+        ixy="8.05787556448484E-13"
+        ixz="9.13275008053385E-13"
+        iyy="8.07147396496025E-09"
+        iyz="1.28152628023355E-12"
+        izz="8.07148645937271E-09" />
+    </inertial>
+    <visual>
+      <origin
+        xyz="0 0 0"
+        rpy="0 0 0" />
+      <geometry>
+        <mesh
+          filename="${mesh_path}camera_infra1_frame.STL" />
+      </geometry>
+      <material
+        name="">
+        <color
+          rgba="0.792156862745098 0.819607843137255 0.933333333333333 1" />
+      </material>
+    </visual>
+    <collision>
+      <origin
+        xyz="0 0 0"
+        rpy="0 0 0" />
+      <geometry>
+        <mesh
+          filename="${mesh_path}camera_infra1_frame.STL" />
+      </geometry>
+    </collision>
+  </link>
+  <joint
+    name="camera_ir_frame"
     type="fixed">
     <origin
@@ -92,78 +145,25 @@
       rpy="0 0 0" />
     <parent
-      link="camera_link" />
-    <child
-      link="camera_botter_screw_frame" />
-    <axis
-      xyz="0 0 0" />
-  </joint>
-  <link
-    name="camera_infra1_frame">
-    <inertial>
-      <origin
-        xyz="-0.000620201436687004 -1.61358465547434E-08 -1.50984520398332E-07"
-        rpy="0 0 0" />
-      <mass
-        value="0.000453168343720438" />
-      <inertia
-        ixx="4.34107789199216E-09"
-        ixy="-3.70099015891851E-13"
-        ixz="-1.46784711283119E-13"
-        iyy="4.84012228066652E-09"
-        iyz="2.0076254107311E-14"
-        izz="4.84044599033091E-09" />
-    </inertial>
-    <visual>
-      <origin
-        xyz="0 0 0"
-        rpy="0 0 0" />
-      <geometry>
-        <mesh
-          filename="${mesh_path}camera_infra1_frame.STL" />
-      </geometry>
-      <material
-        name="">
-        <color
-          rgba="0.792156862745098 0.819607843137255 0.933333333333333 1" />
-      </material>
-    </visual>
-    <collision>
-      <origin
-        xyz="0 0 0"
-        rpy="0 0 0" />
-      <geometry>
-        <mesh
-          filename="${mesh_path}camera_infra1_frame.STL" />
-      </geometry>
-    </collision>
-  </link>
-  <joint
-    name="camera_infra1_frame"
-    type="fixed">
-    <origin
-      xyz="0.01491 -0.025 0.0125"
-      rpy="0 0 0" />
-    <parent
-      link="camera_botter_screw_frame" />
-    <child
-      link="camera_infra1_frame" />
-    <axis
-      xyz="0 0 0" />
-  </joint>
-  <link
-    name="camera_infra1_optical_frame">
-    <inertial>
-      <origin
-        xyz="1.61358465547434E-08 1.50984520398324E-07 -0.000620201436687004"
-        rpy="0 0 0" />
-      <mass
-        value="0.000453168343720438" />
-      <inertia
-        ixx="4.84012228066652E-09"
-        ixy="2.00762541073067E-14"
-        ixz="3.70099015891915E-13"
-        iyy="4.84044599033091E-09"
-        iyz="1.46784711283141E-13"
-        izz="4.34107789199216E-09" />
+      link="camera_depth_frame" />
+    <child
+      link="camera_ir_frame" />
+    <axis
+      xyz="0 0 0" />
+  </joint>
+  <link
+    name="camera_ir_optical_frame">
+    <inertial>
+      <origin
+        xyz="-5.33451517362171E-07 -6.0879600974216E-07 -0.00168460453866946"
+        rpy="0 0 0" />
+      <mass
+        value="0.000608348661221202" />
+      <inertia
+        ixx="8.07147396496025E-09"
+        ixy="1.28152628023355E-12"
+        ixz="-8.0578755644897E-13"
+        iyy="8.07148645937271E-09"
+        iyz="-9.13275008052949E-13"
+        izz="6.79778952271057E-09" />
     </inertial>
     <visual>
@@ -192,5 +192,5 @@
   </link>
   <joint
-    name="camera_infra1_optical_frame"
+    name="camera_ir_optical_frame"
     type="fixed">
     <origin
@@ -198,7 +198,7 @@
       rpy="-1.5707963267949 0 -1.5707963267949" />
     <parent
-      link="camera_infra1_frame" />
-    <child
-      link="camera_infra1_optical_frame" />
+      link="camera_ir_frame" />
+    <child
+      link="camera_ir_optical_frame" />
     <axis
       xyz="0 0 0" />
@@ -208,37 +208,37 @@
     <inertial>
       <origin
-        xyz="2.29364384785394E-07 -2.11520958501546E-07 -0.00105779474323097"
-        rpy="0 0 0" />
-      <mass
-        value="0.000139779411914196" />
-      <inertia
-        ixx="6.11273726117097E-10"
-        ixy="3.95051289663905E-14"
-        ixz="1.55845266007242E-13"
-        iyy="6.11076547268852E-10"
-        iyz="2.25440284353371E-14"
-        izz="6.69129408711142E-10" />
-    </inertial>
-    <visual>
-      <origin
-        xyz="0 0 0"
-        rpy="0 0 0" />
-      <geometry>
-        <mesh
-          filename="${mesh_path}camera_color_frame.STL" />
-      </geometry>
-      <material
-        name="">
-        <color
-          rgba="0.792156862745098 0.819607843137255 0.933333333333333 1" />
-      </material>
-    </visual>
-    <collision>
-      <origin
-        xyz="0 0 0"
-        rpy="0 0 0" />
-      <geometry>
-        <mesh
-          filename="${mesh_path}camera_color_frame.STL" />
+        xyz="-0.0010912488631539 -4.73353451897057E-07 7.19396296308746E-07"
+        rpy="0 0 0" />
+      <mass
+        value="7.68929599151334E-05" />
+      <inertia
+        ixx="3.55949372682833E-10"
+        ixy="-6.02255513042918E-14"
+        ixz="-1.32613402096388E-13"
+        iyy="2.2724816811302E-10"
+        iyz="-4.27828382910552E-14"
+        izz="2.2743913744705E-10" />
+    </inertial>
+    <visual>
+      <origin
+        xyz="0 0 0"
+        rpy="0 0 0" />
+      <geometry>
+        <mesh
+          filename="${mesh_path}camera_colorl_frame.STL" />
+      </geometry>
+      <material
+        name="">
+        <color
+          rgba="0.792156862745098 0.819607843137255 0.933333333333333 1" />
+      </material>
+    </visual>
+    <collision>
+      <origin
+        xyz="0 0 0"
+        rpy="0 0 0" />
+      <geometry>
+        <mesh
+          filename="${mesh_path}camera_colorl_frame.STL" />
       </geometry>
     </collision>
@@ -248,55 +248,108 @@
     type="fixed">
     <origin
-      xyz="0.01682 0.010995 0.012505"
+      xyz="0.0025420000310987234 -0.01850000023841858 0"
+      rpy="0 0 0" />
+    <parent
+      link="camera_depth_frame" />
+    <child
+      link="camera_color_frame" />
+    <axis
+      xyz="0 0 0" />
+  </joint>
+  <link
+    name="camera_color_optical_frame">
+    <inertial>
+      <origin
+        xyz="4.73353451897057E-07 -7.19396296308746E-07 -0.0010912488631539"
+        rpy="0 0 0" />
+      <mass
+        value="7.68929599151334E-05" />
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
File: orbbec_description/urdf/gemini2.urdf.xacro (robot description, xacro)
@@ -3,25 +3,25 @@
      Commit Version: 1.6.0-4-g7f85cfe  Build Version: 1.6.7995.38578
      For more information, please see http://wiki.ros.org/sw_urdf_exporter -->
-<robot xmlns:xacro="http://ros.org/wiki/xacro" name="astra2">
-    <xacro:property name="mesh_path" value="package://orbbec_description/meshes/astra2/" />
+<robot xmlns:xacro="http://ros.org/wiki/xacro" name="gemini2">
+    <xacro:property name="mesh_path" value="package://orbbec_description/meshes/gemini2/" />
   <link
     name="camera_link">
     <inertial>
       <origin
-        xyz="-0.0160938085585399 -0.00100885505248632 0.0279919581775268"
-        rpy="0 0 0" />
-      <mass
-        value="0.0101524380243699" />
-      <inertia
-        ixx="1.69184979927567E-05"
-        ixy="-8.18066547859061E-09"
-        ixz="-1.27426373196599E-09"
-        iyy="7.7096717121366E-07"
-        iyz="1.08838945581987E-08"
-        izz="1.61801971464778E-05" />
-    </inertial>
-    <visual>
-      <origin
-        xyz="0 0 0"
+        xyz="0.0027714370634978 -9.29434319373592E-06 0.0128014057830239"
+        rpy="0 0 0" />
+      <mass
+        value="0.0186201988654731" />
+      <inertia
+        ixx="1.38952652762223E-05"
+        ixy="-4.88105621547421E-09"
+        ixz="1.98670223779875E-08"
+        iyy="1.7072236178685E-06"
+        iyz="-8.49860443053716E-09"
+        izz="1.31795237727551E-05" />
+    </inertial>
+    <visual>
+      <origin
+        xyz="-0.01491 -0.025 -0.0125"
         rpy="0 0 0" />
       <geometry>
@@ -32,5 +32,5 @@
         name="">
         <color
-          rgba="0.827450980392157 0.698039215686274 0.490196078431373 1" />
+          rgba="0.792156862745098 0.819607843137255 0.933333333333333 1" />
       </material>
     </visual>
@@ -46,45 +46,310 @@
   </link>
   <link
-    name="camera_bottom_screw_frame">
-    <inertial>
-      <origin
-        xyz="-0.00635589512085941 1.59480886486103E-08 0.0118534361269284"
-        rpy="0 0 0" />
-      <mass
-        value="0.00583601107155577" />
-      <inertia
-        ixx="3.65092579901689E-06"
-        ixy="-5.00479838523244E-12"
-        ixz="7.68810468643615E-07"
-        iyy="2.03966087595316E-06"
-        iyz="6.18841137398479E-13"
-        izz="3.65126403038314E-06" />
-    </inertial>
-    <visual>
-      <origin
-        xyz="0 0 0"
-        rpy="0 0 0" />
-      <geometry>
-        <mesh
-          filename="${mesh_path}camera_bottom_screw_frame.STL" />
-      </geometry>
-      <material
-        name="">
-        <color
-          rgba="0.266666666666667 0.266666666666667 0.266666666666667 1" />
-      </material>
-    </visual>
-    <collision>
-      <origin
-        xyz="0 0 0"
-        rpy="0 0 0" />
-      <geometry>
-        <mesh
-          filename="${mesh_path}camera_bottom_screw_frame.STL" />
-      </geometry>
-    </collision>
-  </link>
-  <joint
-    name="camera_bottom_screw_frame"
+    name="camera_botter_screw_frame">
+    <inertial>
+      <origin
+        xyz="0.00255175353418556 -0.00123907270798541 0.0118889783016768"
+        rpy="0 0 0" />
+      <mass
+        value="0.00564464822744556" />
+      <inertia
+        ixx="3.07688942133184E-06"
+        ixy="-1.84968755859098E-08"
+        ixz="-9.2787127214088E-09"
+        iyy="2.27625032346061E-07"
+        iyz="1.65176768024159E-08"
+        izz="2.93984854119768E-06" />
+    </inertial>
+    <visual>
+      <origin
+        xyz="0 0 0"
+        rpy="0 0 0" />
+      <geometry>
+        <mesh
+          filename="${mesh_path}camera_botter_screw_frame.STL" />
+      </geometry>
+      <material
+        name="">
+        <color
+          rgba="0.792156862745098 0.819607843137255 0.933333333333333 1" />
+      </material>
+    </visual>
+    <collision>
+      <origin
+        xyz="0 0 0"
+        rpy="0 0 0" />
+      <geometry>
+        <mesh
+          filename="${mesh_path}camera_botter_screw_frame.STL" />
+      </geometry>
+    </collision>
+  </link>
+  <joint
+    name="camera_botter_screw_frame"
+    type="fixed">
+    <origin
+      xyz="-0.01491 -0.025 -0.0125"
+      rpy="0 0 0" />
+    <parent
+      link="camera_link" />
+    <child
+      link="camera_botter_screw_frame" />
+    <axis
+      xyz="0 0 0" />
+  </joint>
+  <link
+    name="camera_right_ir_frame">
+    <inertial>
+      <origin
+        xyz="-0.000620201436687004 -1.61358465547434E-08 -1.50984520398332E-07"
+        rpy="0 0 0" />
+      <mass
+        value="0.000453168343720438" />
+      <inertia
+        ixx="4.34107789199216E-09"
+        ixy="-3.70099015891851E-13"
+        ixz="-1.46784711283119E-13"
+        iyy="4.84012228066652E-09"
+        iyz="2.0076254107311E-14"
+        izz="4.84044599033091E-09" />
+    </inertial>
+    <visual>
+      <origin
+        xyz="0 0 0"
+        rpy="0 0 0" />
+      <geometry>
+        <mesh
+          filename="${mesh_path}camera_infra1_frame.STL" />
+      </geometry>
+      <material
+        name="">
+        <color
+          rgba="0.792156862745098 0.819607843137255 0.933333333333333 1" />
+      </material>
+    </visual>
+    <collision>
+      <origin
+        xyz="0 0 0"
+        rpy="0 0 0" />
+      <geometry>
+        <mesh
+          filename="${mesh_path}camera_infra1_frame.STL" />
+      </geometry>
+    </collision>
+  </link>
+  <joint
+    name="camera_right_ir_frame"
+    type="fixed">
+    <origin
+      xyz="0 -0.05000000074505806 0"
+      rpy="0 0 0" />
+    <parent
+      link="camera_depth_frame" />
+    <child
+      link="camera_right_ir_frame" />
+    <axis
+      xyz="0 0 0" />
+  </joint>
+  <link
+    name="camera_right_ir_optical_frame">
+    <inertial>
+      <origin
+        xyz="1.61358465547434E-08 1.50984520398324E-07 -0.000620201436687004"
+        rpy="0 0 0" />
+      <mass
+        value="0.000453168343720438" />
+      <inertia
+        ixx="4.84012228066652E-09"
+        ixy="2.00762541073067E-14"
+        ixz="3.70099015891915E-13"
+        iyy="4.84044599033091E-09"
+        iyz="1.46784711283141E-13"
+        izz="4.34107789199216E-09" />
+    </inertial>
+    <visual>
+      <origin
+        xyz="0 0 0"
+        rpy="0 0 0" />
+      <geometry>
+        <mesh
+          filename="${mesh_path}camera_infra1_optical_frame.STL" />
+      </geometry>
+      <material
+        name="">
+        <color
+          rgba="0.792156862745098 0.819607843137255 0.933333333333333 1" />
+      </material>
+    </visual>
+    <collision>
+      <origin
+        xyz="0 0 0"
+        rpy="0 0 0" />
+      <geometry>
+        <mesh
+          filename="${mesh_path}camera_infra1_optical_frame.STL" />
+      </geometry>
+    </collision>
+  </link>
+  <joint
+    name="camera_right_ir_optical_frame"
+    type="fixed">
+    <origin
+      xyz="0 0 0"
+      rpy="-1.5707963267949 0 -1.5707963267949" />
+    <parent
+      link="camera_right_ir_frame" />
+    <child
+      link="camera_right_ir_optical_frame" />
+    <axis
+      xyz="0 0 0" />
+  </joint>
+  <link
+    name="camera_color_frame">
+    <inertial>
+      <origin
+        xyz="2.29364384785394E-07 -2.11520958501546E-07 -0.00105779474323097"
+        rpy="0 0 0" />
+      <mass
+        value="0.000139779411914196" />
+      <inertia
+        ixx="6.11273726117097E-10"
+        ixy="3.95051289663905E-14"
+        ixz="1.55845266007242E-13"
+        iyy="6.11076547268852E-10"
+        iyz="2.25440284353371E-14"
+        izz="6.69129408711142E-10" />
+    </inertial>
+    <visual>
+      <origin
+        xyz="0 0 0"
+        rpy="0 0 0" />
+      <geometry>
+        <mesh
+          filename="${mesh_path}camera_color_frame.STL" />
+      </geometry>
+      <material
+        name="">
+        <color
+          rgba="0.792156862745098 0.819607843137255 0.933333333333333 1" />
+      </material>
+    </visual>
+    <collision>
+      <origin
+        xyz="0 0 0"
+        rpy="0 0 0" />
+      <geometry>
+        <mesh
+          filename="${mesh_path}camera_color_frame.STL" />
+      </geometry>
+    </collision>
+  </link>
+  <joint
+    name="camera_color_frame"
+    type="fixed">
+    <origin
+      xyz="0.0019099999917671084 -0.01400499977171421 4.999999873689376e-06"
+      rpy="0 0 0" />
+    <parent
+      link="camera_depth_frame" />
+    <child
+      link="camera_color_frame" />
+    <axis
+      xyz="0 0 0" />
+  </joint>
+  <link
+    name="camera_color_optical_frame">
+    <inertial>
+      <origin
+        xyz="2.29364384785394E-07 -2.11520958501541E-07 -0.00105779474323097"
+        rpy="0 0 0" />
+      <mass
+        value="0.000139779411914196" />
+      <inertia
+        ixx="6.11273726117097E-10"
+        ixy="3.95051289663901E-14"
+        ixz="1.55845266007242E-13"
+        iyy="6.11076547268852E-10"
+        iyz="2.25440284353391E-14"
+        izz="6.69129408711142E-10" />
+    </inertial>
+    <visual>
+      <origin
+        xyz="0 0 0"
+        rpy="0 0 0" />
+      <geometry>
+        <mesh
+          filename="${mesh_path}camera_color_optical_frame.STL" />
+      </geometry>
+      <material
+        name="">
+        <color
+          rgba="0.792156862745098 0.819607843137255 0.933333333333333 1" />
+      </material>
+    </visual>
+    <collision>
+      <origin
+        xyz="0 0 0"
+        rpy="0 0 0" />
+      <geometry>
+        <mesh
+          filename="${mesh_path}camera_color_optical_frame.STL" />
+      </geometry>
+    </collision>
+  </link>
+  <joint
+    name="camera_color_optical_frame"
+    type="fixed">
+    <origin
+      xyz="0 0 0"
+      rpy="-1.5707963267949 0 -1.5707963267949" />
+    <parent
+      link="camera_color_frame" />
+    <child
+      link="camera_color_optical_frame" />
+    <axis
+      xyz="0 0 0" />
+  </joint>
+  <link
+    name="camera_left_ir_frame">
+    <inertial>
+      <origin
+        xyz="-0.000620201436687001 -1.6135846551274E-08 -1.50984520410662E-07"
+        rpy="0 0 0" />
+      <mass
+        value="0.000453168343720439" />
+      <inertia
+        ixx="4.34107789199216E-09"
+        ixy="-3.70099015888916E-13"
+        ixz="-1.46784711288897E-13"
+        iyy="4.84012228066651E-09"
+        iyz="2.0076254105875E-14"
+        izz="4.8404459903309E-09" />
+    </inertial>
+    <visual>
+      <origin
+        xyz="0 0 0"
+        rpy="0 0 0" />
+      <geometry>
+        <mesh
+          filename="${mesh_path}camera_infra2_frame.STL" />
+      </geometry>
+      <material
+        name="">
+        <color
+          rgba="0.792156862745098 0.819607843137255 0.933333333333333 1" />
+      </material>
+    </visual>
+    <collision>
+      <origin
+        xyz="0 0 0"
+        rpy="0 0 0" />
+      <geometry>
+        <mesh
+          filename="${mesh_path}camera_infra2_frame.STL" />
+      </geometry>
+    </collision>
+  </link>
+  <joint
+    name="camera_left_ir_frame"
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
File: orbbec_description/urdf/test_gemini2L.urdf.xacro (robot description, xacro)
@@ -3,6 +3,6 @@
      Commit Version: 1.6.0-4-g7f85cfe  Build Version: 1.6.7995.38578
      For more information, please see http://wiki.ros.org/sw_urdf_exporter -->
-<robot name="gemini_335" xmlns:xacro="http://ros.org/wiki/xacro">
-    <xacro:include filename="gemini_335_336.urdf.xacro"/>
+<robot name="gemini2L" xmlns:xacro="http://ros.org/wiki/xacro">
+    <xacro:include filename="gemini2L.urdf.xacro"/>
     <!-- Define a virtual root link -->
   <link name="base_link"/>
@@ -11,5 +11,5 @@
     <parent link="base_link"/>
     <child link="camera_link"/>
-    <origin xyz="0 0 0" rpy="0 0 0"/>
+    <origin xyz="0.01033 0.05 0.0145" rpy="0 0 0"/>
   </joint>
 </robot>
