Commit message: Rebase from 'upstream'

File: orbbec_description/urdf/test_gemini335L.urdf.xacro (robot description, xacro)
@@ -3,6 +3,6 @@
      Commit Version: 1.6.0-4-g7f85cfe  Build Version: 1.6.7995.38578
      For more information, please see http://wiki.ros.org/sw_urdf_exporter -->
-<robot name="gemini336L" xmlns:xacro="http://ros.org/wiki/xacro">
-    <xacro:include filename="gemini335L_336L.urdf.xarco"/>
+<robot name="gemini335L" xmlns:xacro="http://ros.org/wiki/xacro">
+    <xacro:include filename="gemini335L_336L.urdf.xacro"/>
     <!-- Define a virtual root link -->
   <link name="base_link"/>
@@ -11,5 +11,5 @@
     <parent link="base_link"/>
     <child link="camera_link"/>
-    <origin xyz="0 0 0" rpy="0 0 0"/>
+    <origin xyz="0.011715 0.0475 0.014311" rpy="0 0 0"/>
   </joint>
 </robot>

File: orbbec_description/urdf/test_gemini335Le.urdf.xacro (robot description, xacro)
@@ -3,6 +3,6 @@
      Commit Version: 1.6.0-4-g7f85cfe  Build Version: 1.6.7995.38578
      For more information, please see http://wiki.ros.org/sw_urdf_exporter -->
-<robot name="gemini2" xmlns:xacro="http://ros.org/wiki/xacro">
-    <xacro:include filename="gemini2.urdf.xarco"/>
+<robot name="gemini335Le" xmlns:xacro="http://ros.org/wiki/xacro">
+    <xacro:include filename="gemini335Le.urdf.xacro"/>
     <!-- Define a virtual root link -->
   <link name="base_link"/>
@@ -11,5 +11,5 @@
     <parent link="base_link"/>
     <child link="camera_link"/>
-    <origin xyz="0 0 0" rpy="0 0 0"/>
+    <origin xyz="0.034005 0.0475 0.014048" rpy="0 0 0"/>
   </joint>
 </robot>

File: orbbec_description/urdf/test_gemini335Lg.urdf.xacro (robot description, xacro)
@@ -3,6 +3,6 @@
      Commit Version: 1.6.0-4-g7f85cfe  Build Version: 1.6.7995.38578
      For more information, please see http://wiki.ros.org/sw_urdf_exporter -->
-<robot name="gemini_336" xmlns:xacro="http://ros.org/wiki/xacro">
-    <xacro:include filename="gemini_335_336.urdf.xacro"/>
+<robot name="gemini335Lg" xmlns:xacro="http://ros.org/wiki/xacro">
+    <xacro:include filename="gemini335Lg.urdf.xacro"/>
     <!-- Define a virtual root link -->
   <link name="base_link"/>
@@ -11,5 +11,5 @@
     <parent link="base_link"/>
     <child link="camera_link"/>
-    <origin xyz="0 0 0" rpy="0 0 0"/>
+    <origin xyz="0.0117149999999995 0.0475 0.0143111800025738" rpy="0 0 0"/>
   </joint>
 </robot>

File: orbbec_description/urdf/test_gemini_335.urdf.xacro (robot description, xacro)
@@ -3,6 +3,6 @@
      Commit Version: 1.6.0-4-g7f85cfe  Build Version: 1.6.7995.38578
      For more information, please see http://wiki.ros.org/sw_urdf_exporter -->
-<robot name="gemini335Lg" xmlns:xacro="http://ros.org/wiki/xacro">
-    <xacro:include filename="gemini335Lg.urdf.xacro"/>
+<robot name="gemini_335" xmlns:xacro="http://ros.org/wiki/xacro">
+    <xacro:include filename="gemini_335_336.urdf.xacro"/>
     <!-- Define a virtual root link -->
   <link name="base_link"/>
@@ -11,5 +11,5 @@
     <parent link="base_link"/>
     <child link="camera_link"/>
-    <origin xyz="0 0 0" rpy="0 0 0"/>
+    <origin xyz="0.01587 0.025 0.0125" rpy="0 0 0"/>
   </joint>
 </robot>

File: orbbec_description/urdf/test_gemini_336.urdf.xacro (robot description, xacro)
@@ -3,6 +3,6 @@
      Commit Version: 1.6.0-4-g7f85cfe  Build Version: 1.6.7995.38578
      For more information, please see http://wiki.ros.org/sw_urdf_exporter -->
-<robot name="gemini335L" xmlns:xacro="http://ros.org/wiki/xacro">
-    <xacro:include filename="gemini335L_336L.urdf.xarco"/>
+<robot name="gemini_336" xmlns:xacro="http://ros.org/wiki/xacro">
+    <xacro:include filename="gemini_335_336.urdf.xacro"/>
     <!-- Define a virtual root link -->
   <link name="base_link"/>
@@ -11,5 +11,5 @@
     <parent link="base_link"/>
     <child link="camera_link"/>
-    <origin xyz="0 0 0" rpy="0 0 0"/>
+    <origin xyz="0.01587 0.025 0.0125" rpy="0 0 0"/>
   </joint>
 </robot>
